File: Z88 Flash KiCad/z88-flash-mod.kicad_pcb (KiCad board)
At the start: 4 copper layers, 50.5 x 52.5 mm, 12 parts, among them J1 Conn_Z88, U1 AM29F800B [JEDEC 1024k x8 / 5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, U2 HY628400A LLG-70, U3 HY628400A LLG-70, U4 74LS139

Commit message: tweaks
Parts:
- JP1: value 512k -> 512KB RAM
Changed lines of the file:
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@@
 			)
 		)
-		(property "Datasheet" ""
+		(property "Datasheet" "~"
 			(at 0 0 90)
 			(layer "F.Fab")
@@
 		)
 		(property ki_fp_filters "C_*")
-		(sheetname "Root")
+		(sheetname "/")
 		(sheetfile "z88-flash-mod.kicad_sch")
 		(attr smd)
@@
 			)
 		)
-		(property "Datasheet" ""
+		(property "Datasheet" "~"
 			(at 0 0 90)
 			(layer "F.Fab")
@@
 		)
 		(property ki_fp_filters "C_*")
-		(sheetname "Root")
+		(sheetname "/")
 		(sheetfile "z88-flash-mod.kicad_sch")
 		(attr smd)
@@
 		)
 		(property "Datasheet" "https://www.alliancememory.com/wp-content/uploads/pdf/AS6C4008.pdf"
-			(at 0 0 270)
+			(at 0 0 90)
 			(layer "F.Fab")
 			(hide yes)
@@
 			)
 		)
-		(property "Description" ""
-			(at 0 0 270)
+		(property "Description" "512K x 8 Low Power CMOS RAM, DIP-32"
+			(at 0 0 90)
 			(layer "F.Fab")
 			(hide yes)
@@
 		)
 		(property ki_fp_filters "DIP*W15.24mm*")
-		(sheetname "Root")
+		(sheetname "/")
 		(sheetfile "z88-flash-mod.kicad_sch")
 		(attr smd)
@@
 		)
 		(property ki_fp_filters "DIP?16*")
-		(sheetname "Root")
+		(sheetname "/")
 		(sheetfile "z88-flash-mod.kicad_sch")
 		(attr smd)
@@
 			)
 		)
-		(property "Datasheet" ""
+		(property "Datasheet" "~"
 			(at 0 0 0)
 			(layer "F.Fab")
@@
 		)
 		(property ki_fp_filters "LED* LED_SMD:* LED_THT:*")
-		(sheetname "Root")
+		(sheetname "/")
 		(sheetfile "z88-flash-mod.kicad_sch")
 		(attr smd)
@@
 		)
 		(property ki_fp_filters "TSOP*18.*12*P0.5mm*")
-		(sheetname "Root")
+		(sheetname "/")
 		(sheetfile "z88-flash-mod.kicad_sch")
 		(attr smd)
@@
 			)
 		)
-		(property "Value" "512k"
+		(property "Value" "512KB RAM"
 			(at 0 1.9 90)
 			(layer "F.SilkS")
@@
 			)
 		)
-		(property "Datasheet" ""
+		(property "Datasheet" "~"
 			(at 0 0 90)
 			(layer "F.Fab")
@@
 			)
 		)
-		(property "Description" "Jumper, 2-pole, open"
+		(property "Description" ""
 			(at 0 0 90)
 			(layer "F.Fab")
@@
 			)
 		)
-		(sheetfile "connector.kicad_sch")
+		(property ki_fp_filters "Jumper* TestPoint*2Pads* TestPoint*Bridge*")
+		(sheetname "/")
+		(sheetfile "z88-flash-mod.kicad_sch")
 		(attr exclude_from_pos_files)
 		(fp_line
@@
 			)
 		)
-		(property "Datasheet" ""
+		(property "Datasheet" "~"
 			(at 0 0 0)
 			(layer "F.Fab")
@@
 		)
 		(property ki_fp_filters "R_*")
-		(sheetname "Root")
+		(sheetname "/")
 		(sheetfile "z88-flash-mod.kicad_sch")
 		(attr smd)
@@
 			)
 		)
-		(property "Datasheet" ""
+		(property "Datasheet" "~"
 			(at 0 0 90)
 			(layer "F.Fab")
@@
 		)
 		(property ki_fp_filters "C_*")
-		(sheetname "Root")
+		(sheetname "/")
 		(sheetfile "z88-flash-mod.kicad_sch")
 		(attr smd)
@@
 			)
 		)
-		(property "Datasheet" ""
+		(property "Datasheet" "~"
 			(at 0 0 0)
 			(layer "F.Fab")
@@
 		)
 		(property ki_fp_filters "Connector*:*2x??x*mm* Connector*:*2x???Pitch*")
-		(sheetname "Root")
+		(sheetname "/")
 		(sheetfile "z88-flash-mod.kicad_sch")
 		(attr through_hole)
@@
 			)
 		)
-		(property "Description" ""
+		(property "Description" "512K x 8 Low Power CMOS RAM, DIP-32"
 			(at 0 0 270)
 			(layer "F.Fab")
@@
 		)
 		(property ki_fp_filters "DIP*W15.24mm*")
-		(sheetname "Root")
+		(sheetname "/")
 		(sheetfile "z88-flash-mod.kicad_sch")
 		(attr smd)
@@
 		(layer "F.Cu")
 		(name "$teardrop_padvia$")
-		(hatch full 0.1)
+		(hatch none 0.1)
 		(priority 30000)
 		(attr
