File: Z88 Flash KiCad/z88-flash-mod.kicad_sch (KiCad schematic)
At the start: 11 parts, among them J1 Conn_Z88, U1 AM29F800B [JEDEC 1024k x8 / 5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, U2 HY628400A LLG-70, U3 HY628400A LLG-70, U4 74LS139

Commit message: little tweaks
Parts:
- U2, U3: footprint Package_SO:SSOP-32_11.305x20.495mm_P1.27mm -> Package_DIP:DIP-32_W15.24mm

Commit message: tweaks
Parts:
- J1: symbol connector-rescue:Conn_Z88-Connector -> Z88:Z88_Card
- U2, U3: footprint Package_DIP:DIP-32_W15.24mm -> Package_SO:SSOP-32_11.305x20.495mm_P1.27mm
Connections:
- net GND: no longer J1.15n (Pin_53), J1.17 (GND)
- net VCC: no longer J1.21 (Pin_21)
- net WEL renamed ~{WE}
- no-connect marks 37 -> 2
